File: electronics/adder.sch (KiCad schematic (older format))
At the start: 16 parts, among them U1 74LS386, U15 74LS08, U2 74LS386, U3 74LS283, U36 74LS02, U37 74LS08, U4 74LS283, U5 74LS245

Commit message: Some initial electronics design
Not everything done yet, just committing to show progress and to get the changes out of the way.
Parts:
- removed ACC_LATCH1: 74LS377, Package_DIP:DIP-20_W7.62mm, symbol 74xx:74LS377
- removed C20, C21, C22, C23, C24, C25, C26: 0.1µF, Capacitor_THT:CP_Radial_D4.0mm_P1.50mm, symbol Device:C
- removed U1, U2: 74LS386, Package_DIP:DIP-14_W7.62mm, symbol 74xx:74LS386
- removed U15, U37: 74LS08, Package_DIP:DIP-14_W7.62mm, symbol 74xx:74LS08
- removed U3, U4: 74LS283, Package_DIP:DIP-16_W7.62mm, symbol 74xx:74LS283
- removed U36: 74LS02, Package_DIP:DIP-14_W7.62mm, symbol 74xx:74LS02
- removed U5: 74LS245, Package_DIP:DIP-20_W7.62mm, symbol 74xx:74LS245
- added U34, U35: 74LS86, symbol 74xx:74LS86
- added U36, U37: 74LS283, symbol 74xx:74LS283
Connections:
- net +5V: now also U34.14 (VCC), U35.14 (VCC), U36.16 (VCC), U37.16 (VCC)
- net GND: now also U34.7 (GND), U35.7 (GND), U36.8 (GND), U37.8 (GND)
- net SUB: now also U34.1, U34.12, U34.4, U34.9, U35.1, U35.12, U35.4, U35.9, U36.7 (C0)
- new net: U34.11, U36.11 (B4)
- new net: U34.8, U36.15 (B3)
- new net: U34.6, U36.2 (B2)
- new net: U34.3, U36.6 (B1)
- new net: U36.9 (C4), U37.7 (C0)
- new net: U35.3, U37.6 (B1)
- new net: U35.6, U37.2 (B2)
- new net: U35.8, U37.15 (B3)
- new net: U35.11, U37.11 (B4)
- new net A0: U36.5 (A1)
- new net A1: U36.3 (A2)
- new net A2: U36.14 (A3)
- new net A3: U36.12 (A4)
- new net A4: U37.5 (A1)
- new net A5: U37.3 (A2)
- new net A6: U37.14 (A3)
- new net A7: U37.12 (A4)
- new net B0: U34.2
- new net B1: U34.5
- new net B2: U34.10
- new net B3: U34.13
- new net B4: U35.2
- new net B5: U35.5
- new net B6: U35.10
- new net B7: U35.13
- new net CARRY: U37.9 (C4)
- new net S0: U36.4 (S1)
- new net S1: U36.1 (S2)
- new net S2: U36.13 (S3)
- new net S3: U36.10 (S4)
- new net S4: U37.4 (S1)
- new net S5: U37.1 (S2)
- new net S6: U37.13 (S3)
- new net S7: U37.10 (S4)
Other:
- note removed: "Accumulator Latch Register"
- note removed: "Adder"
- note removed: "Carry\nFlag"
- note removed: "D[0..7] Inverter"
- note removed: "Zero Flag"
