File: electronics/flag.sch (KiCad schematic (older format))
At the start: 2 parts, among them U35 74LS377

Commit message: Some initial electronics design
Not everything done yet, just committing to show progress and to get the changes out of the way.
Parts:
- removed C19: 0.1µF, Capacitor_THT:CP_Radial_D4.0mm_P1.50mm, symbol Device:C
- removed U35: 74LS377, Package_DIP:DIP-20_W7.62mm, symbol 74xx:74LS377
- added U11: 74LS08, symbol 74xx:74LS08
- added U40: 74LS273, symbol 74xx:74LS273
Connections:
- net +5V: now also U40.20 (VCC)
- net C_IN: now also U40.4 (D1)
- net C_OUT: now also U40.5 (Q1)
- net GND: now also U40.10 (GND)
- net Z_IN: now also U40.3 (D0)
- net Z_OUT: now also U40.2 (Q0)
- net ~CLK: now also U11.10
- new net: U11.8, U40.11 (Cp)
- new net LOAD: U11.9
- new net ~RESET: U40.1 (~Mr)
Changed lines of the file:
@@
 $Descr A4 11693 8268
 encoding utf-8
-Sheet 9 14
-Title "Flag Register"
-Date "2019-08-10"
-Rev "1"
-Comp "Zac Garby"
+Sheet 13 14
+Title ""
+Date ""
+Rev ""
+Comp ""
 Comment1 ""
 Comment2 ""
@@
 $EndDescr
 $Comp
-L 74xx:74LS377 U?
-U 1 1 5DB73BD8
-P 5450 3400
-AR Path="/5D483C2B/5DB73BD8" Ref="U?"  Part="1"
-AR Path="/5D48A331/5DB73BD8" Ref="U?"  Part="1"
-AR Path="/5DB6B499/5DB73BD8" Ref="U35"  Part="1"
-F 0 "U35" H 5500 4150 50  0000 L CNN
-F 1 "74LS377" H 5500 4050 50  0000 L CNN
-F 2 "Package_DIP:DIP-20_W7.62mm" H 5450 3400 50  0001 C CNN
-F 3 "http://www.ti.com/lit/gpn/sn74LS377" H 5450 3400 50  0001 C CNN
-	1    5450 3400
+L power:+5V #PWR097
+U 1 1 5D98B5F4
+P 5200 2500
+F 0 "#PWR097" H 5200 2350 50  0001 C CNN
+F 1 "+5V" H 5215 2675 50  0000 C CNN
+F 2 "" H 5200 2500 50  0001 C CNN
+F 3 "" H 5200 2500 50  0001 C CNN
+	1    5200 2500
+	1    0    0    -1
+$EndComp
+$Comp
+L power:GND #PWR098
+U 1 1 5D98B714
+P 5200 4100
+F 0 "#PWR098" H 5200 3850 50  0001 C CNN
+F 1 "GND" H 5205 3925 50  0000 C CNN
+F 2 "" H 5200 4100 50  0001 C CNN
+F 3 "" H 5200 4100 50  0001 C CNN
+	1    5200 4100
+	1    0    0    -1
+$EndComp
+Text GLabel 4700 3800 3    50   Input ~ 0
+~RESET
+$Comp
+L 74xx:74LS08 U11
+U 3 1 5D98DF05
+P 4250 3700
+F 0 "U11" H 4250 3400 50  0000 C CNN
+F 1 "74LS08" H 4250 3500 50  0000 C CNN
+F 2 "" H 4250 3700 50  0001 C CNN
+F 3 "http://www.ti.com/lit/gpn/sn74LS08" H 4250 3700 50  0001 C CNN
+	3    4250 3700
 	1    0    0    -1
 $EndComp
 Wire Wire Line
-	4950 3800 4900 3800
-Wire Wire Line
-	4950 3900 4900 3900
-Text HLabel 4900 3950 0    50   Input ~ 0
-~IN
+	4550 3700 4700 3700
+Text GLabel 3950 3800 0    50   Input ~ 0
+~CLK
+Text HLabel 3950 3600 0    50   Input ~ 0
+LOAD
+Text HLabel 4700 2800 0    50   Input ~ 0
+Z_IN
+Text HLabel 4700 2900 0    50   Input ~ 0
+C_IN
+Text HLabel 5700 2800 2    50   Output ~ 0
+Z_OUT
+Text HLabel 5700 2900 2    50   Output ~ 0
+C_OUT
+NoConn ~ 4700 3000
+NoConn ~ 4700 3100
 $Comp
-L power:+5V #PWR?
-U 1 1 5DB73BE2
-P 5450 2600
-AR Path="/5D483C2B/5DB73BE2" Ref="#PWR?"  Part="1"
-AR Path="/5D48A331/5DB73BE2" Ref="#PWR?"  Part="1"
-AR Path="/5DB6B499/5DB73BE2" Ref="#PWR067"  Part="1"
-F 0 "#PWR067" H 5450 2450 50  0001 C CNN
-F 1 "+5V" H 5465 2773 50  0000 C CNN
-F 2 "" H 5450 2600 50  0001 C CNN
-F 3 "" H 5450 2600 50  0001 C CNN
-	1    5450 2600
+L 74xx:74LS273 U40
+U 1 1 5D989E0E
+P 5200 3300
+F 0 "U40" H 5250 4050 50  0000 L CNN
+F 1 "74LS273" H 5250 3950 50  0000 L CNN
+F 2 "" H 5200 3300 50  0001 C CNN
+F 3 "http://www.ti.com/lit/gpn/sn74LS273" H 5200 3300 50  0001 C CNN
+	1    5200 3300
 	1    0    0    -1
 $EndComp
-$Comp
-L power:GND #PWR?
-U 1 1 5DB73BE8
-P 5450 4200
-AR Path="/5D483C2B/5DB73BE8" Ref="#PWR?"  Part="1"
-AR Path="/5D48A331/5DB73BE8" Ref="#PWR?"  Part="1"
-AR Path="/5DB6B499/5DB73BE8" Ref="#PWR068"  Part="1"
-F 0 "#PWR068" H 5450 3950 50  0001 C CNN
-F 1 "GND" H 5455 4027 50  0000 C CNN
-F 2 "" H 5450 4200 50  0001 C CNN
-F 3 "" H 5450 4200 50  0001 C CNN
-	1    5450 4200
-	1    0    0    -1
-$EndComp
-Wire Wire Line
-	4950 3000 4400 3000
-Wire Wire Line
-	4400 2900 4950 2900
-Wire Wire Line
-	6500 3000 5950 3000
-Wire Wire Line
-	5950 2900 6500 2900
-NoConn ~ 4950 3100
-NoConn ~ 4950 3200
-NoConn ~ 4950 3300
-NoConn ~ 4950 3400
-NoConn ~ 4950 3500
-NoConn ~ 4950 3600
-NoConn ~ 5950 3100
-NoConn ~ 5950 3200
-NoConn ~ 5950 3300
-NoConn ~ 5950 3400
-NoConn ~ 5950 3500
-NoConn ~ 5950 3600
-Text HLabel 4400 2900 0    50   Input ~ 0
-Z_IN
-Text HLabel 4400 3000 0    50   Input ~ 0
-C_IN
-Text HLabel 6500 2900 2    50   Output ~ 0
-Z_OUT
-Text HLabel 6500 3000 2    50   Output ~ 0
-C_OUT
-Text GLabel 4900 3800 0    50   Input ~ 0
-~CLK
-Wire Wire Line
-	4900 3900 4900 3950
-$Comp
-L power:+5V #PWR?
-U 1 1 5D59B542
-P 7750 3050
-AR Path="/5D59B542" Ref="#PWR?"  Part="1"
-AR Path="/5DB6B499/5D59B542" Ref="#PWR0127"  Part="1"
-F 0 "#PWR0127" H 7750 2900 50  0001 C CNN
-F 1 "+5V" H 7765 3223 50  0000 C CNN
-F 2 "" H 7750 3050 50  0001 C CNN
-F 3 "" H 7750 3050 50  0001 C CNN
-	1    7750 3050
-	1    0    0    -1
-$EndComp
-$Comp
-L Device:C C?
-U 1 1 5D59B548
-P 7750 3300
-AR Path="/5D59B548" Ref="C?"  Part="1"
-AR Path="/5DB6B499/5D59B548" Ref="C19"  Part="1"
-F 0 "C19" H 7865 3346 50  0000 L CNN
-F 1 "0.1µF" H 7865 3255 50  0000 L CNN
-F 2 "Capacitor_THT:CP_Radial_D4.0mm_P1.50mm" H 7788 3150 50  0001 C CNN
-F 3 "~" H 7750 3300 50  0001 C CNN
-	1    7750 3300
-	1    0    0    -1
-$EndComp
-$Comp
-L power:GND #PWR?
-U 1 1 5D59B54E
-P 7750 3550
-AR Path="/5D59B54E" Ref="#PWR?"  Part="1"
-AR Path="/5DB6B499/5D59B54E" Ref="#PWR0128"  Part="1"
-F 0 "#PWR0128" H 7750 3300 50  0001 C CNN
-F 1 "GND" H 7755 3377 50  0000 C CNN
-F 2 "" H 7750 3550 50  0001 C CNN
-F 3 "" H 7750 3550 50  0001 C CNN
-	1    7750 3550
-	1    0    0    -1
-$EndComp
-Wire Wire Line
-	7750 3550 7750 3450
-Wire Wire Line
-	7750 3150 7750 3050
+NoConn ~ 4700 3200
+NoConn ~ 4700 3300
+NoConn ~ 4700 3400
+NoConn ~ 4700 3500
+NoConn ~ 5700 3500
+NoConn ~ 5700 3400
+NoConn ~ 5700 3300
+NoConn ~ 5700 3200
+NoConn ~ 5700 3100
+NoConn ~ 5700 3000
 $EndSCHEMATC
