File: electronics/ram.sch (KiCad schematic (older format))
At the start: 5 parts, among them U10 AS6C62256-55PCN, U11 AS6C62256-55PCN, U12 74LS04

Commit message: Some initial electronics design
Not everything done yet, just committing to show progress and to get the changes out of the way.
Parts:
- removed C4, C5: 0.1µF, Capacitor_THT:CP_Radial_D4.0mm_P1.50mm, symbol Device:C
- removed U10, U11: AS6C62256-55PCN, Package_DIP:DIP-28_W15.24mm, symbol misc_components:AS6C62256-55PCN
- removed U12: 74LS04, Package_DIP:DIP-14_W7.62mm, symbol 74xx:74LS04
- added U16: 74LS04, symbol 74xx:74LS04
- added U17, U18: AS6C62256-55PCN, symbol misc_components:AS6C62256-55PCN
- added U19: 74LS245, symbol 74xx:74LS245
Connections:
- net +5V: now also U16.14 (VCC), U17.28 (Vcc), U18.28 (Vcc), U19.20 (VCC)
- net A0: now also U17.10 (A0), U18.10 (A0)
- net A1: now also U17.9 (A1), U18.9 (A1)
- net A10: now also U17.21 (A10), U18.21 (A10)
- net A11: now also U17.23 (A11), U18.23 (A11)
- net A12: now also U17.2 (A12), U18.2 (A12)
- net A13: now also U17.26 (A13), U18.26 (A13)
- net A14: now also U17.1 (A14), U18.1 (A14)
- net A15: now also U16.1, U17.20 (~CE)
- net A2: now also U17.8 (A2), U18.8 (A2)
- net A3: now also U17.7 (A3), U18.7 (A3)
- net A4: now also U17.6 (A4), U18.6 (A4)
- net A5: now also U17.5 (A5), U18.5 (A5)
- net A6: now also U17.4 (A6), U18.4 (A6)
- net A7: now also U17.3 (A7), U18.3 (A7)
- net A8: now also U17.25 (A8), U18.25 (A8)
- net A9: now also U17.24 (A9), U18.24 (A9)
- net D0: now also U19.2 (A0)
- net D1: now also U19.3 (A1)
- net D2: now also U19.4 (A2)
- net D3: now also U19.5 (A3)
- net D4: now also U19.6 (A4)
- net D5: now also U19.7 (A5)
- net D6: now also U19.8 (A6)
- net D7: now also U19.9 (A7)
- net GND: now also U16.7 (GND), U17.14 (GND), U18.14 (GND), U19.10 (GND), U19.19 (CE)
- net ~IN: now also U17.27 (~WE), U18.27 (~WE)
- net ~OUT: now also U17.22 (~OE), U18.22 (~OE), U19.1 (A->B)
- new net: U17.11 (DQ0), U18.11 (DQ0), U19.18 (B0)
- new net: U17.12 (DQ1), U18.12 (DQ1), U19.17 (B1)
- new net: U17.13 (DQ2), U18.13 (DQ2), U19.16 (B2)
- new net: U17.15 (DQ3), U18.15 (DQ3), U19.15 (B3)
- new net: U17.16 (DQ4), U18.16 (DQ4), U19.14 (B4)
- new net: U17.17 (DQ5), U18.17 (DQ5), U19.13 (B5)
- new net: U17.18 (DQ6), U18.18 (DQ6), U19.12 (B6)
- new net: U17.19 (DQ7), U18.19 (DQ7), U19.11 (B7)
- new net: U16.2, U18.20 (~CE)
