File: electronics/register.sch (KiCad schematic (older format))
At the start: 3 parts, among them U6 74LS377, U7 74LS245

Commit message: Some initial electronics design
Not everything done yet, just committing to show progress and to get the changes out of the way.
Parts:
- removed C2: 0.1µF, Capacitor_THT:CP_Radial_D4.0mm_P1.50mm, symbol Device:C
- removed U6: 74LS377, Package_DIP:DIP-20_W7.62mm, symbol 74xx:74LS377
- removed U7: 74LS245, Package_DIP:DIP-20_W7.62mm, symbol 74xx:74LS245
- added U?: 74LS273, symbol 74xx:74LS273
- added U?: 74LS08, symbol 74xx:74LS08
- added U?: 74LS245, symbol 74xx:74LS245
Connections:
- net +5V: now also U?.1 (~Mr), U?.20 (VCC)
- net D0: now also U?.3 (D0)
- net D1: now also U?.4 (D1)
- net D2: now also U?.7 (D2)
- net D3: now also U?.8 (D3)
- net D4: now also U?.13 (D4)
- net D5: now also U?.14 (D5)
- net D6: now also U?.17 (D6)
- net D7: now also U?.18 (D7)
- net GND: now also U?.10 (GND)
- net ~CLK: now also U?.2
- new net: U?.11 (Cp), U?.3
- new net: U?.12 (Q4), U?.6 (A4)
- new net: U?.15 (Q5), U?.7 (A5)
- new net: U?.16 (Q6), U?.8 (A6)
- new net: U?.19 (Q7), U?.9 (A7)
- new net: U?.2 (A0), U?.2 (Q0)
- new net: U?.3 (A1), U?.5 (Q1)
- new net: U?.4 (A2), U?.6 (Q2)
- new net: U?.5 (A3), U?.9 (Q3)
- new net IN: U?.1
